Commit message: fix camera urdf direction

File: omniduino_description/urdf/camera.urdf.xacro (robot description, xacro)
@@ -5,5 +5,5 @@
       <parent link="${parent}"/>
       <child  link="${prefix}_link"/>
-      <origin xyz="${xyz}" rpy="${radians(-90)} 0 ${radians(-90)}"/>
+      <origin xyz="${xyz}" rpy="${radians(-90)} 0 0"/>
     </joint>
     <link name="${prefix}_link"/>
