Commit message: fix urdf

File: omniduino_description/urdf/N20GearedMotor.urdf.xacro (robot description, xacro)
@@ -26,4 +26,5 @@
     <link name="${prefix}_shaft_link">
       <visual><geometry><cylinder radius="0.00125" length="0.014" /></geometry></visual>
+      <collision><geometry><cylinder radius="0.00125" length="0.014" /></geometry></collision>
       <inertial><xacro:cylinder_inertial mass="0.001" radius="0.00125" length="0.014" /></inertial>
     </link>

File: omniduino_description/urdf/mecanum37.urdf.xacro (robot description, xacro)
@@ -13,5 +13,5 @@
       </geometry><material name="black"/></visual>
       <collision><geometry>
-        <cylinder radius="0.005" length="0.024" />
+        <cylinder radius="0.005" length="0.01" />
       </geometry></collision>
       <inertial><xacro:cylinder_inertial mass="0.01" radius="0.009" length="0.024" /></inertial>
@@ -29,4 +29,5 @@
         <cylinder radius="0.017" length="0.005" />
       </geometry><material name="black"/></visual>
+      <inertial><xacro:cylinder_inertial mass="0.0001" radius="0.017" length="0.0381" /></inertial>
     </link>
     <joint name="${prefix}_${inout}_frame" type="fixed">

Commit message: (not work)change param for sim

File: omniduino_description/urdf/N20GearedMotor.urdf.xacro (robot description, xacro)
@@ -34,4 +34,5 @@
       <origin xyz="0.022 0 0" rpy="0 ${pi/2} 0"/>
       <axis xyz="0 0 1"/>
+      <limit velocity="1.0" effort="20000" />
       <dynamics damping="0.001" friction="0.0" />
     </joint>

File: omniduino_description/urdf/main.urdf.xacro (robot description, xacro)
@@ -15,5 +15,5 @@
     <parent link="base_link" />
     <child  link="base_plate_link" />
-    <origin xyz="0 0 0.02" />
+    <origin xyz="0 0 0.01" />
   </joint>
   <gazebo reference="base_plate_link">
@@ -23,5 +23,5 @@
     <visual><geometry><box size="0.031 0.088 0.022" /></geometry><material name="black"/></visual>
     <collision><geometry><box size="0.031 0.088 0.022" /></geometry></collision>
-    <inertial><xacro:box_inertial mass="0.200" height="0.031" width="0.088" depth="0.022"/></inertial>
+    <inertial><xacro:box_inertial mass="0.600" height="0.031" width="0.088" depth="0.022"/></inertial>
   </link>
   <joint name="battery_link_joint" type="fixed">
@@ -71,5 +71,5 @@
     <axis xyz="0 1 0" />
     <limit lower="${-20.0/180.0*pi}" upper="${20.0/180.0*pi}" effort="0.2" velocity="5" />
-    <dynamics damping="0.0" friction="0.0" />
+    <dynamics damping="0.01" friction="0.0" />
   </joint>
   <transmission name="camera_trans">

File: omniduino_description/urdf/sus.urdf.xacro (robot description, xacro)
@@ -11,8 +11,8 @@
       <parent link="${parent}" />
       <child  link="${prefix}_link" />
-      <limit lower="-0.001" upper="0.001" effort="100" velocity="1.0" />
+      <limit lower="-0.002" upper="0.002" effort="100" velocity="1.0" />
       <axis xyz="0 0 1" />
       <origin xyz="${xyz}" rpy="${rpy}" />
-      <dynamics damping="0.001" />
+      <dynamics damping="0.01" />
     </joint>
     <transmission name="${prefix}_trans">

Commit message: change controller&interface

File: omniduino_description/urdf/N20GearedMotor.urdf.xacro (robot description, xacro)
@@ -34,5 +34,4 @@
       <origin xyz="0.022 0 0" rpy="0 ${pi/2} 0"/>
       <axis xyz="0 0 1"/>
-      <limit velocity="1.0" effort="20000" />
       <dynamics damping="0.001" friction="0.0" />
     </joint>
@@ -40,8 +39,8 @@
       <type>transmission_interface/SimpleTransmission</type>
       <joint name="${prefix}_shaft_joint">
-        <hardwareInterface>hardware_interface/VelocityJointInterface</hardwareInterface>
+        <hardwareInterface>hardware_interface/EffortJointInterface</hardwareInterface>
       </joint>
       <actuator name="${prefix}_shaft_motor">
-        <hardwareInterface>hardware_interface/VelocityJointInterface</hardwareInterface>
+        <hardwareInterface>hardware_interface/EffortJointInterface</hardwareInterface>
         <mechanicalReduction>1</mechanicalReduction>
       </actuator>
