Commit message: (work done) change param for sim

File: omniduino_description/urdf/main.urdf.xacro (robot description, xacro)
@@ -10,5 +10,5 @@
     <visual><geometry><box size="0.114 0.062 0.005" /></geometry><material name="black"/></visual>
     <collision><geometry><box size="0.114 0.062 0.005" /></geometry></collision>
-    <inertial><xacro:box_inertial mass="0.030" height="0.114" width="0.062" depth="0.005"/></inertial>
+    <inertial><xacro:box_inertial mass="1.0" height="0.114" width="0.062" depth="0.005"/></inertial>
   </link>
   <joint name="base_plate_link" type="fixed">
@@ -23,5 +23,5 @@
     <visual><geometry><box size="0.031 0.088 0.022" /></geometry><material name="black"/></visual>
     <collision><geometry><box size="0.031 0.088 0.022" /></geometry></collision>
-    <inertial><xacro:box_inertial mass="0.600" height="0.031" width="0.088" depth="0.022"/></inertial>
+    <inertial><xacro:box_inertial mass="10.0" height="0.031" width="0.088" depth="0.022"/></inertial>
   </link>
   <joint name="battery_link_joint" type="fixed">
@@ -36,5 +36,5 @@
     <visual><geometry><box size="0.114 0.114 0.01" /></geometry><material name="black"/></visual>
     <collision><geometry><box size="0.085 0.085 0.01" /></geometry></collision>
-    <inertial><xacro:box_inertial mass="0.050" height="0.114" width="0.114" depth="0.01"/></inertial>
+    <inertial><xacro:box_inertial mass="0.50" height="0.114" width="0.114" depth="0.01"/></inertial>
   </link>
   <joint name="controll_board_link_joint" type="fixed">
@@ -49,5 +49,5 @@
     <visual><geometry><box size="0.0273 0.0325 0.012" /></geometry><material name="black"/></visual>
     <collision><geometry><box size="0.0273 0.0325 0.012" /></geometry></collision>
-    <inertial><xacro:box_inertial mass="0.035" height="0.0273" width="0.0325" depth="0.012"/></inertial>
+    <inertial><xacro:box_inertial mass="1.0" height="0.0273" width="0.0325" depth="0.012"/></inertial>
   </link>
   <joint name="servo_link_joint" type="fixed">
@@ -63,5 +63,5 @@
     <visual><geometry><box size="0.030 0.035 0.035" /></geometry><material name="white"/></visual>
     <collision><geometry><box size="0.030 0.035 0.035" /></geometry></collision>
-    <inertial><xacro:box_inertial mass="0.020" height="0.030" width="0.035" depth="0.035"/></inertial>
+    <inertial><xacro:box_inertial mass="0.1" height="0.030" width="0.035" depth="0.035"/></inertial>
   </link>
   <joint name="camera_base_link_joint" type="revolute">

File: omniduino_description/urdf/mecanum37.urdf.xacro (robot description, xacro)
@@ -18,5 +18,5 @@
       <child  link="${prefix}_shaft" />
       <origin xyz="${joint_xyz}" rpy="${joint_rpy}" />
-      <dynamics damping="0.001" friction="0.0" />
+      <dynamics damping="0.00001" friction="0.0" />
     </joint>
   </xacro:macro>
@@ -45,5 +45,5 @@
           <mesh filename="package://omniduino_description/meshes/ffbarrel.stl" />
       </geometry></collision>
-      <inertial><xacro:cylinder_inertial mass="0.01225" radius="0.00956" length="0.0381" /></inertial>
+      <inertial><xacro:cylinder_inertial mass="0.01225" radius="0.01" length="0.0261" /></inertial>
     </link>
     <joint name="${prefix}_barrel${num}_joint" type="continuous">
@@ -52,5 +52,5 @@
       <origin rpy="0 ${pi/4*rot} ${radians(dir)+pi/2}" xyz="${0.012975*cos(radians(dir))} ${0.012975*sin(radians(dir))} 0"/>
       <axis xyz="1 0 0"/>
-      <dynamics damping="0.001"  friction="0.0"/>
+      <dynamics damping="0.00001"  friction="0.0"/>
     </joint>
     <gazebo reference="${prefix}_barrel${num}_link">
