Commit message: fix robots model direction

File: omniduino_description/robots/omniduino.urdf.xacro (robot description, xacro)
@@ -10,17 +10,17 @@
   <xacro:macro name="wheel_module" params="number rot parent_link joint_xyz joint_rpy">
     <xacro:N20_motor prefix="motor${number}" parent_link="${parent_link}" joint_xyz="${joint_xyz}" joint_rpy="${joint_rpy}"/>
-    <xacro:mecanum_wheel prefix="wheel${number}" parent_link="motor${number}_shaft_link" rot="${rot}" joint_xyz="0 0 0.012" joint_rpy="0 0 0"/>
+    <xacro:mecanum_wheel prefix="wheel${number}" parent_link="motor${number}_shaft_link" rot="${rot}" joint_xyz="0 0 0.008" joint_rpy="0 0 0"/>
   </xacro:macro>
-  <xacro:wheel_module number="1" rot=" 1" parent_link="base_plate_link" joint_xyz=" 0.0155  0.038 0.00825" joint_rpy="0 0 0" />
-  <xacro:wheel_module number="2" rot="-1" parent_link="base_plate_link" joint_xyz=" 0.0155 -0.038 0.00825" joint_rpy="0 0 0" />
-  <xacro:wheel_module number="3" rot="-1" parent_link="base_plate_link" joint_xyz="-0.0155  0.038 0.00825" joint_rpy="0 0 ${pi}" />
-  <xacro:wheel_module number="4" rot=" 1" parent_link="base_plate_link" joint_xyz="-0.0155 -0.038 0.00825" joint_rpy="0 0 ${pi}" />
-  <xacro:gazebo_light_sensor name="front"  parent="controll_borad_link" xyz=" 0     0.05 0" direction="0" />
-  <xacro:gazebo_light_sensor name="fleft"  parent="controll_borad_link" xyz="-0.05  0.05 0" direction="${ pi/4}" />
-  <xacro:gazebo_light_sensor name="fright" parent="controll_borad_link" xyz=" 0.05  0.05 0" direction="${-pi/4}" />
-  <xacro:gazebo_light_sensor name="rleft"  parent="controll_borad_link" xyz="-0.05 -0.05 0" direction="${ pi/4*3}" />
-  <xacro:gazebo_light_sensor name="rright" parent="controll_borad_link" xyz=" 0.05 -0.05 0" direction="${-pi/4*3}" />
+  <xacro:wheel_module number="1" rot="-1" parent_link="base_plate_link" joint_xyz=" 0.038  0.0155 0.00825" joint_rpy="0 0 ${ pi/2}" />
+  <xacro:wheel_module number="2" rot=" 1" parent_link="base_plate_link" joint_xyz="-0.038  0.0155 0.00825" joint_rpy="0 0 ${ pi/2}" />
+  <xacro:wheel_module number="3" rot=" 1" parent_link="base_plate_link" joint_xyz=" 0.038 -0.0155 0.00825" joint_rpy="0 0 ${-pi/2}" />
+  <xacro:wheel_module number="4" rot="-1" parent_link="base_plate_link" joint_xyz="-0.038 -0.0155 0.00825" joint_rpy="0 0 ${-pi/2}" />
+  <xacro:gazebo_light_sensor name="front"  parent="controll_borad_link" xyz=" 0.05     0  0" direction="${-pi/2}" />
+  <xacro:gazebo_light_sensor name="fleft"  parent="controll_borad_link" xyz=" 0.05  0.05  0" direction="${-pi/4}" />
+  <xacro:gazebo_light_sensor name="fright" parent="controll_borad_link" xyz=" 0.05 -0.05  0" direction="${-pi/4*3}" />
+  <xacro:gazebo_light_sensor name="rleft"  parent="controll_borad_link" xyz="-0.05  0.05  0" direction="${ pi/4}" />
+  <xacro:gazebo_light_sensor name="rright" parent="controll_borad_link" xyz="-0.05 -0.05  0" direction="${ pi/4*3}" />
   <xacro:imu_macro parent="controll_borad_link" prefix="imu" xyz="0 0 0" />
-  <xacro:camera_macro parent="camera_link" prefix="camera1" xyz="0 0.015 0" />
+  <xacro:camera_macro parent="camera_link" prefix="camera1" xyz="0.015 0 0" />
   <gazebo>
     <plugin name="gazebo_ros_control" filename="libgazebo_ros_control.so">

File: omniduino_description/urdf/camera.urdf.xacro (robot description, xacro)
@@ -5,5 +5,5 @@
       <parent link="${parent}"/>
       <child  link="${prefix}_link"/>
-      <origin xyz="${xyz}" rpy="${radians(-90)} 0 0"/>
+      <origin xyz="${xyz}" rpy="${radians(-90)} 0 ${radians(-90)}"/>
     </joint>
     <link name="${prefix}_link"/>

File: omniduino_description/urdf/main.urdf.xacro (robot description, xacro)
@@ -8,7 +8,7 @@
   </xacro:macro>
   <link name="base_plate_link">
-    <visual><geometry><box size="0.062 0.114 0.005" /></geometry><material name="black"/></visual>
-    <collision><geometry><box size="0.062 0.114 0.005" /></geometry></collision>
-    <inertial><xacro:box_inertial mass="0.030" height="0.062" width="0.114" depth="0.005"/></inertial>
+    <visual><geometry><box size="0.114 0.062 0.005" /></geometry><material name="black"/></visual>
+    <collision><geometry><box size="0.114 0.062 0.005" /></geometry></collision>
+    <inertial><xacro:box_inertial mass="0.030" height="0.114" width="0.062" depth="0.005"/></inertial>
   </link>
   <joint name="base_plate_link" type="fixed">
@@ -21,7 +21,7 @@
   </gazebo>
   <link name="battery_link">
-    <visual><geometry><box size="0.088 0.031 0.022" /></geometry><material name="black"/></visual>
-    <collision><geometry><box size="0.088 0.031 0.022" /></geometry></collision>
-    <inertial><xacro:box_inertial mass="0.200" height="0.088" width="0.031" depth="0.022"/></inertial>
+    <visual><geometry><box size="0.031 0.088 0.022" /></geometry><material name="black"/></visual>
+    <collision><geometry><box size="0.031 0.088 0.022" /></geometry></collision>
+    <inertial><xacro:box_inertial mass="0.200" height="0.031" width="0.088" depth="0.022"/></inertial>
   </link>
   <joint name="battery_link_joint" type="fixed">
@@ -35,5 +35,5 @@
   <link name="controll_borad_link">
     <visual><geometry><box size="0.114 0.114 0.01" /></geometry><material name="black"/></visual>
-    <collision><geometry><box size="0.114 0.114 0.01" /></geometry></collision>
+    <collision><geometry><box size="0.085 0.085 0.01" /></geometry></collision>
     <inertial><xacro:box_inertial mass="0.050" height="0.114" width="0.114" depth="0.01"/></inertial>
   </link>
@@ -47,12 +47,12 @@
   </gazebo>
   <link name="servo_link">
-    <visual><geometry><box size="0.0325 0.0273 0.012" /></geometry><material name="black"/></visual>
-    <collision><geometry><box size="0.0325 0.0273 0.012" /></geometry></collision>
-    <inertial><xacro:box_inertial mass="0.035" height="0.0325" width="0.0273" depth="0.012"/></inertial>
+    <visual><geometry><box size="0.0273 0.0325 0.012" /></geometry><material name="black"/></visual>
+    <collision><geometry><box size="0.0273 0.0325 0.012" /></geometry></collision>
+    <inertial><xacro:box_inertial mass="0.035" height="0.0273" width="0.0325" depth="0.012"/></inertial>
   </link>
   <joint name="servo_link_joint" type="fixed">
     <parent link="controll_borad_link" />
     <child  link="servo_link" />
-    <origin xyz="0 0.01 0.011" />
+    <origin xyz="0.01 0 0.011" />
   </joint>
   <gazebo reference="servo_link">
@@ -61,13 +61,13 @@
   <link name="camera_base_link"/>
   <link name="camera_link">
-    <visual><geometry><box size="0.035 0.030 0.035" /></geometry><material name="white"/></visual>
-    <collision><geometry><box size="0.035 0.030 0.035" /></geometry></collision>
-    <inertial><xacro:box_inertial mass="0.020" height="0.035" width="0.030" depth="0.035"/></inertial>
+    <visual><geometry><box size="0.030 0.035 0.035" /></geometry><material name="white"/></visual>
+    <collision><geometry><box size="0.030 0.035 0.035" /></geometry></collision>
+    <inertial><xacro:box_inertial mass="0.020" height="0.030" width="0.035" depth="0.035"/></inertial>
   </link>
   <joint name="camera_base_link_joint" type="revolute">
     <parent link="servo_link" />
     <child  link="camera_base_link" />
-    <origin xyz="0 0.005 0" />
-    <axis xyz="1 0 0" />
+    <origin xyz="0.005 0 0" />
+    <axis xyz="0 1 0" />
     <limit lower="${-20.0/180.0*pi}" upper="${20.0/180.0*pi}" effort="0.2" velocity="5" />
     <dynamics damping="0.0" friction="0.0" />

File: omniduino_description/urdf/mecanum37.urdf.xacro (robot description, xacro)
@@ -12,7 +12,4 @@
         <cylinder radius="0.005" length="0.024" />
       </geometry><material name="black"/></visual>
-      <collision><geometry>
-        <cylinder radius="0.005" length="0.01" />
-      </geometry></collision>
       <inertial><xacro:cylinder_inertial mass="0.01" radius="0.009" length="0.024" /></inertial>
     </link>
@@ -75,6 +72,6 @@
   <xacro:macro name="mecanum_wheel" params="prefix parent_link rot joint_xyz joint_rpy">
     <xacro:wheel_shaft prefix="${prefix}" parent_link="${parent_link}" joint_xyz="${joint_xyz}" joint_rpy="${joint_rpy}"/>
-    <xacro:wheel_frame prefix="${prefix}" inout="inside"  to_shaft_length=" 0.0135" />
-    <xacro:wheel_frame prefix="${prefix}" inout="outside" to_shaft_length="-0.0135" />
+    <xacro:wheel_frame prefix="${prefix}" inout="inside"  to_shaft_length=" 0.01" />
+    <xacro:wheel_frame prefix="${prefix}" inout="outside" to_shaft_length="-0.01" />
     <xacro:barrels prefix="${prefix}" rot="${rot}" />
   </xacro:macro>
